File: psk-modulator/psk-modulator.kicad_sch (KiCad schematic)
At the start: 23 parts, among them J3 RFOUT, J4 DSOP, J5 IBBN, J6 IBBP, J7 QBBN, J8 QBBP, U1 ADL5375, U2 ADF4351

Commit message: rocktrack
Parts:
- removed J5: IBBN, Connector_Coaxial:SMA_Samtec_SMA-J-P-H-ST-EM1_EdgeMount, symbol Connector:Conn_Coaxial_Small
- removed J6: IBBP, Connector_Coaxial:SMA_Samtec_SMA-J-P-H-ST-EM1_EdgeMount, symbol Connector:Conn_Coaxial_Small
- removed J7: QBBN, Connector_Coaxial:SMA_Samtec_SMA-J-P-H-ST-EM1_EdgeMount, symbol Connector:Conn_Coaxial_Small
- removed J8: QBBP, Connector_Coaxial:SMA_Samtec_SMA-J-P-H-ST-EM1_EdgeMount, symbol Connector:Conn_Coaxial_Small
- removed U2: ADF4351, Package_CSP:LFCSP-32-1EP_5x5mm_P0.5mm_EP3.25x3.25mm, symbol Timer_PLL:ADF4351
- added C10, C11, C12, C13: C, Capacitor_SMD:C_0402_1005Metric, symbol Device:C_Small
- added J1: LON, Connector_Coaxial:SMA_Samtec_SMA-J-P-H-ST-EM1_EdgeMount, symbol Connector:Conn_Coaxial_Small
- added J2: LOP, Connector_Coaxial:SMA_Samtec_SMA-J-P-H-ST-EM1_EdgeMount, symbol Connector:Conn_Coaxial_Small
- added L1, L2, L3, L4: L, Inductor_SMD:L_0402_1005Metric, symbol Device:L_Small
- added U3: AD9709, Package_QFP:LQFP-48_7x7mm_P0.5mm, symbol TxDAC:AD9709
Connections:
- net GND: now also J1.2 (Ext), J2.2 (Ext)
- net QBBNF: now reaches R6.2
- net QBBNF: now also U1.9 (QBBN), C13.2, L4.1; no longer U1.10 (QBBP)
- net IBBNF: now reaches R5.2
- net IBBNF: now also U1.22 (IBBN), C10.2, L2.1; no longer U1.21 (IBBP)
- net IBBPF: now reaches R5.1
- net IBBPF: now also U1.21 (IBBP), C10.1, L1.2; no longer U1.22 (IBBN)
- net QBBPF: now reaches R6.1
- net QBBPF: now also U1.10 (QBBP), C13.1, L3.2; no longer U1.9 (QBBN)
- net LOP: now reaches C8.1, R4.2
- net LOP: now also J2.1 (In)
- net LON: now reaches C8.2, R3.2
- net LON: now also J1.1 (In)
- new net: U3.10 (NC), U3.11 (NC), U3.12 (NC), U3.13 (NC), U3.14 (NC), U3.31 (NC), U3.32 (NC), U3.33 (NC), U3.34 (NC), U3.35 (NC), U3.36 (NC), U3.9 (NC)
- new net: U3.15 (DGND), U3.21 (DGND)
- new net DVCC: U3.16 (DVCC), U3.22 (DVCC)
- new net IBBN: C11.2, L2.2, U3.45 (IOUTB1)
- new net IBBP: C11.1, L1.1, U3.46 (IOUTA1)
- new net QBBN: C12.2, L4.2, U3.40 (IOUTB2)
- new net QBBP: C12.1, L3.1, U3.39 (IOUTA2)
Other:
- moved on the sheet: C1, C2, C3, C4, C5, C6, C7, C8, C9, J3, J4, R1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
