File: psk-modulator/psk-modulator.kicad_sch (KiCad schematic)
At the start: 29 parts, among them J1 LON, J2 LOP, J3 RFOUT, J4 DSOP, U1 ADL5375, U3 AD9709

Commit message: stuff
Parts:
- removed J1: LON, Connector_Coaxial:SMA_Samtec_SMA-J-P-H-ST-EM1_EdgeMount, symbol Connector:Conn_Coaxial_Small
- removed J2: LOP, Connector_Coaxial:SMA_Samtec_SMA-J-P-H-ST-EM1_EdgeMount, symbol Connector:Conn_Coaxial_Small
- added C14, C15: 100n, symbol Device:C_Small
- added FB1: FerriteBead_Small, symbol Device:FerriteBead_Small
- added R7, R8: 2k, Inductor_SMD:L_0402_1005Metric, symbol Device:R_Small
- added U2: ADF4351, Package_CSP:LFCSP-32-1EP_5x5mm_P0.5mm_EP3.25x3.25mm, symbol Timer_PLL:ADF4351
- C6, C7, C8: footprint Capacitor_SMD:C_0603_1608Metric -> Capacitor_SMD:C_0402_1005Metric
- R1, R2, R3, R4: footprint Resistor_SMD:R_0603_1608Metric -> Inductor_SMD:L_0402_1005Metric
Connections:
- net DVCC is gone; now on net +3V3: U3.16 (DVCC), U3.22 (DVCC)
- net GND: now also U3.15 (DGND), U3.21 (DGND), U3.38 (AGND), C14.1, C15.1, R7.2, R8.2, U2.11 (AGNDVCO), U2.18 (AGNDVCO), U2.21 (AGNDVCO), U2.27 (DGND), U2.31 (SDGND), U2.33 (EP), U2.8 (CPGND), U2.9 (AGND)
- net LON: now also U2.13 (RF_OUT_A-)
- net LOP: now also U2.12 (RF_OUT_A+)
- net DB7I: now reaches U3.1 (DB7P1)
- net DB6I: now reaches U3.2 (DB6P1)
- net DB7Q: now reaches U3.23 (DB7P2)
- net DB6Q: now reaches U3.24 (DB6P2)
- net DB5Q: now reaches U3.25 (DB5P2)
- net DB4Q: now reaches U3.26 (DB4P2)
- net DB3Q: now reaches U3.27 (DB3P2)
- net DB2Q: now reaches U3.28 (DB2P2)
- net DB1Q: now reaches U3.29 (DB1P2)
- net DB5I: now reaches U3.3 (DB5P1)
- net DB0Q: now reaches U3.30 (DB0P2)
- net DB4I: now reaches U3.4 (DB4P1)
- net at U3.41 (FSADJ2): now also R7.1
- net at U3.44 (FSADJ1): now also R8.1
- net DB3I: now reaches U3.5 (DB3P1)
- net DB2I: now reaches U3.6 (DB2P1)
- net DB1I: now reaches U3.7 (DB1P1)
- net DB0I: now reaches U3.8 (DB0P1)
