File: ublox_max_breakout/ublox_max_breakout.kicad_pcb (KiCad board)
At the start: 2 copper layers, 19.5 x 26.6 mm, 14 parts, among them J1 U.Fl, J2 SMA, J3 Conn_01x08, U1 MAX-M10S

Commit message: stuff
Parts:
- added PPS: PPS, LED_SMD:LED_0603_1608Metric, F.Cu at (163.3, 110.8)
- added PWR: PWR, LED_SMD:LED_0603_1608Metric, F.Cu at (161.6, 110.8)
- added R3: 270, Resistor_SMD:R_0603_1608Metric, F.Cu at (161.9, 114.6)
- added R4: 270, Resistor_SMD:R_0603_1608Metric, F.Cu at (163.4, 114.6)
- moved C4 1.55 mm to (159.5, 115.7)
- moved C3 1.55 mm to (159.5, 114.1)
- moved JP1 1.30 mm to (162.5, 103.3), turned to 180 degrees
- moved BT1 0.10 mm to (152.5, 116.1)
Connections:
- J3 pad 8: GND -> /PPS
Routing:
- net /PPS: track 0.00 -> 28.5 mm, vias 0 -> 2
- net +3V3: track 35.7 -> 43.4 mm
- net Net-(LED2-A): track 0.00 -> 2.50 mm
- net Net-(LED1-A): track 0.00 -> 2.40 mm
- net Net-(JP1-B): track 9.51 -> 10.3 mm
- net GND: vias 1 -> 70
- removed copper zone on F.Cu, net +3V3
Other:
- board text added: "3V3"
- board text added: "MCzop 2026"
- board text added: "PPS"
- board text added: "RST"
- board text added: "RXD"
- board text added: "SCL"
- board text added: "SDA"
- board text added: "TXD"
- board text added: "Ublox MAX breakout Rev. 1.0"
