File: ublox_max_breakout/ublox_max_breakout.kicad_sch (KiCad schematic)
At the start: 14 parts, among them J1 U.Fl, J2 SMA, J3 Conn_01x08, U1 MAX-M10S

Commit message: stuff
Parts:
- added LED1: PWR, LED_SMD:LED_0603_1608Metric, symbol Device:LED
- added LED2: PPS, LED_SMD:LED_0603_1608Metric, symbol Device:LED
- added R3, R4: 270, Resistor_SMD:R_0603_1608Metric, symbol Device:R_Small
Connections:
- net +3V3: now also R3.1
- net GND: now also LED1.1 (K), LED2.1 (K); no longer J3.8 (Pin_8)
- net PPS: now also J3.8 (Pin_8), R4.1
- new net: LED1.2 (A), R3.2
- new net: LED2.2 (A), R4.2
