File: bpsk-modulator/bpsk-modulator.kicad_sch (KiCad schematic)
At the start: 13 parts, among them J1 RF_OUT, U1 ADE-1, U2 ADF4351, U3 AD9708AR

Commit message: stuff 2
Parts:
- removed A1: RaspberryPi_Pico, Module:RaspberryPi_Pico_Common_SMD, symbol MCU_Module:RaspberryPi_Pico
- removed TR1: JA4220, RF_Components:JA4220, symbol Transformer:TR60_IC
- removed U1: ADE-1, RF_Mini-Circuits:Mini-Circuits_CD542_LandPatternPL-052, symbol RF_Mixer:ADE-6
- removed U2: ADF4351, Package_CSP:LFCSP-32-1EP_5x5mm_P0.5mm_EP3.25x3.25mm, symbol Timer_PLL:ADF4351
- added C10, C17, C19, C5: 1n, Capacitor_SMD:C_0603_1608Metric_Pad1.08x0.95mm_HandSolder, symbol Device:C_Small
- added C11, C12, C13, C14, C15, C24, C25, C29, C31: 100n, Capacitor_SMD:C_0603_1608Metric_Pad1.08x0.95mm_HandSolder, symbol Device:C_Small
- added C16: 22p, Capacitor_SMD:C_0603_1608Metric_Pad1.08x0.95mm_HandSolder, symbol Device:C_Small
- added C18: 10n, Capacitor_SMD:C_0603_1608Metric_Pad1.08x0.95mm_HandSolder, symbol Device:C_Small
- added C20: 1u, Capacitor_SMD:C_0603_1608Metric_Pad1.08x0.95mm_HandSolder, symbol Device:C_Small
- added C21, C22, C23, C26, C27, C28, C30: 4.7u, Capacitor_SMD:C_0603_1608Metric_Pad1.08x0.95mm_HandSolder, symbol Device:C_Small
- added C6, C7, C8, C9: C, Capacitor_SMD:C_0603_1608Metric_Pad1.08x0.95mm_HandSolder, symbol Device:C_Small
- added FB1: 1000, Inductor_SMD:L_0603_1608Metric, symbol Device:FerriteBead_Small
- added J2: LO_IN, Connector_Coaxial:SMA_Samtec_SMA-J-P-H-ST-EM1_EdgeMount, symbol Connector:Conn_Coaxial_Small
- added J3: Header Connector, Connector_PinHeader_2.54mm:PinHeader_2x12_P2.54mm_Vertical, symbol Connector_Generic:Conn_02x12_Odd_Even
- added L4, L5, L6, L7: L, Inductor_SMD:L_0603_1608Metric, symbol Device:L_Small
- added R1, R3, R4: 50, Resistor_SMD:R_0603_1608Metric_Pad0.98x0.95mm_HandSolder, symbol Device:R_Small
- added R10, R11, R9: R, Resistor_SMD:R_0603_1608Metric_Pad0.98x0.95mm_HandSolder, symbol Device:R_Small
- added R12: 39, Resistor_SMD:R_0603_1608Metric_Pad0.98x0.95mm_HandSolder, symbol Device:R_Small
- added R13: 270k, Resistor_SMD:R_0603_1608Metric_Pad0.98x0.95mm_HandSolder, symbol Device:R_Small
- added R14: 100k, Resistor_SMD:R_0603_1608Metric_Pad0.98x0.95mm_HandSolder, symbol Device:R_Small
- added R2: 2k, Resistor_SMD:R_0603_1608Metric_Pad0.98x0.95mm_HandSolder, symbol Device:R_Small
- added R5, R6: 1k, Resistor_SMD:R_0603_1608Metric_Pad0.98x0.95mm_HandSolder, symbol Device:R_Small
- added R7, R8: 499, Resistor_SMD:R_0603_1608Metric_Pad0.98x0.95mm_HandSolder, symbol Device:R_Small
- added U1: SYM-2500+, RF_Mini-Circuits:Mini-Circuits_TTT167_LandPatternPL-079, symbol RF_Mixers:SYM-2500+
- added U3: AD8055, Package_SO:SOIC-8_3.9x4.9mm_P1.27mm, symbol Amplifier_Operational:LMH6609MA
- added U4: GALI-1, Package_TO_SOT_SMD:SOT-89-3, symbol RF_Amplifier:GALI-1
- added U5: LM27761, Package_SON:WSON-8-1EP_2x2mm_P0.5mm_EP0.9x1.6mm, symbol Regulator_SwitchedCapacitor:LM27761
- added U6: AMS1117-3.3, Package_TO_SOT_SMD:SOT-223-3_TabPin2, symbol Regulator_Linear:AMS1117-3.3
- renumbered U3 to U2
Connections:
- net GND: now also U2.16 (REFLO), U2.20 (ACOM), U2.26 (DCOM), C10.2, C11.1, C12.2, C14.1, C15.2, C18.1, C21.1, C22.1, C23.1, C24.2, C25.1, C26.1, C27.1, C28.1, C29.2, C30.1, C31.2, C5.1, C6.2, C7.2, C8.2, C9.2, J2.2 (Ext), J3.1 (Pin_1), J3.2 (Pin_2), J3.23 (Pin_23), J3.24 (Pin_24), R10.1, R11.1, R14.1, R2.2, R3.1, R4.1, R7.2, U1.4 (GND), U4.2 (GND), U5.2 (GND), U5.9 (PAD), U6.1 (GND)
- net DB7: now reaches U2.1 (DB7)
- net DB7: now also J3.17 (Pin_17), J3.18 (Pin_18)
- net at U2.17 (REFIO): now also C15.1
- net at U2.18 (FS_ADJ): now also R2.1
- net at U2.19 (COMP1): now also C13.1
- net DB6: now reaches U2.2 (DB6)
- net DB6: now also J3.15 (Pin_15), J3.16 (Pin_16)
- net OUTN: now reaches U2.21 (IOUTB)
- net OUTN: now also C16.2, R4.2, R5.2
- net OUTP: now reaches U2.22 (IOUTA)
- net OUTP: now also C16.1, R3.2, R6.1
- net at U2.23 (COMP2): now also C12.1
- net VDDA: now reaches U2.24 (AVDD)
- net VDDA: now also C13.2, C14.2, C26.2, FB1.2
- net +3V3: now reaches U2.27 (DVDD)
- net +3V3: now also C11.2, C27.2, C28.2, C29.1, FB1.1, U6.2 (VO)
- net BCLK: now reaches U2.28 (Clock)
- net BCLK: now also J3.19 (Pin_19), J3.20 (Pin_20)
- net DB5: now reaches U2.3 (DB5)
- net DB5: now also J3.13 (Pin_13), J3.14 (Pin_14)
- net DB4: now reaches U2.4 (DB4)
- net DB4: now also J3.11 (Pin_11), J3.12 (Pin_12)
- net DB3: now reaches U2.5 (DB3)
- net DB3: now also J3.10 (Pin_10), J3.9 (Pin_9)
- net DB2: now reaches U2.6 (DB2)
- net DB2: now also J3.7 (Pin_7), J3.8 (Pin_8)
- net DB1: now reaches U2.7 (DB1)
- net DB1: now also J3.5 (Pin_5), J3.6 (Pin_6)
- net DB0: now reaches U2.8 (DB0)
- net DB0: now also J3.3 (Pin_3), J3.4 (Pin_4)
- net at C1.1, L1.1: now also U1.1 (RF)
- new net: R10.2, R9.2, U1.2 (LO)
- new net: C9.1, L6.2, U1.3 (IF)
- new net: C17.1, J2.1 (In)
- new net: R13.2, R14.2, U5.5 (VFB)
- new net: C19.1, L7.1, U4.3
- new net: C18.2, L7.2, R12.2
- new net: C17.2, U4.1
- new net: C7.1, L4.2, L5.1
- new net: C22.2, U5.3 (CPOUT)
- new net: C20.1, U5.7 (C-)
- new net: C20.2, U5.8 (C+)
- new net: C6.1, L4.1, R1.2
- new net: R6.2, R8.1, U3.2 (-)
- new net: C19.2, R11.2, R9.1
- new net: R5.1, R7.1, U3.3 (+)
- new net: C8.1, L5.2, L6.1
- new net +5V: C21.2, C25.2, C30.2, C31.1, C5.2, J3.21 (Pin_21), J3.22 (Pin_22), R12.1, U3.7 (V+), U5.1 (VIN), U5.6 (EN), U6.3 (VI)
- new net -5V: C10.1, C23.2, C24.1, R13.1, U3.4 (V-), U5.4 (VOUT)
- new net OUT: R1.1, R8.2, U3.6
- no-connect marks 2 -> 1
Other:
- moved on the sheet: C1, C2, C3, C4, J1, L1, L2, L3, U2
