File: pha-202+_amplifier_2/pha-202+_amplifier.kicad_pcb (KiCad board)
At the start: 2 copper layers, 16 parts, among them J1 SMA, J2 SMA, J3 PWR, U1 PHA-202+

Commit message: h
Parts:
- removed H5: MountingHole_Pad, MountingHole:MountingHole_3.2mm_M3_DIN965_Pad_TopBottom
- H1, H2, H3, H4: value MountingHole_Pad -> M2.5; footprint MountingHole:MountingHole_3.2mm_M3_DIN965_Pad_TopBottom -> MountingHole:MountingHole_2.7mm_M2.5_DIN965_Pad_TopBottom
- J3: footprint Connector_PinHeader_2.54mm:PinHeader_1x02_P2.54mm_Vertical -> TerminalBlock_Phoenix:TerminalBlock_Phoenix_MKDS-1,5-2_1x02_P5.00mm_Horizontal
- moved H3 65.5 mm to (123.0, 117.0)
- moved H1 62.7 mm to (123.0, 93.0)
- moved J2 42.5 mm to (157.9, 107.2)
- moved C1 35.3 mm to (130.0, 107.2)
- moved H4 31.7 mm to (157.0, 117.0)
- moved J1 28.3 mm to (122.1, 107.2), turned to 180 degrees
- moved H2 28.0 mm to (157.0, 93.0)
- moved L1 24.1 mm to (147.6, 105.2), turned to 180 degrees
- moved C2 22.6 mm to (152.2, 107.2)
- moved PWR 14.8 mm to (150.9, 91.6), turned to 180 degrees
- moved C3 14.5 mm to (147.6, 99.8), turned to 180 degrees
- moved C4 13.8 mm to (147.6, 101.5), turned to 180 degrees
- moved J3 13.4 mm to (141.9, 94.7), turned to 180 degrees
- moved U1 12.0 mm to (137.9, 107.8)
- moved R1 7.82 mm to (147.2, 91.6), turned to 180 degrees
- renumbered D1 to PWR
Routing:
- net VCC: track 0.00 -> 26.2 mm
- net Net-(U1-RFO): track 0.00 -> 10.7 mm
- net Net-(J1-In): track 0.00 -> 7.10 mm
- net Net-(J2-In): track 0.00 -> 4.95 mm
- net Net-(U1-RFIN): track 0.00 -> 4.30 mm
- net Net-(D1-A): track 0.00 -> 2.00 mm
- net GND: vias 0 -> 296
- added copper zone on B.Cu, net GND
- added copper zone on F.Cu, net GND
Other:
- board outline added: 40 x 30 mm
- board text added: "12V MAX!"
- board text added: "GND"
- board text added: "MCzop 2026"
- board text added: "PHA-202+ Amplifier"
- board text added: "RFIN"
- board text added: "RFOUT"
- board text added: "VCC"
