File: pha-202+_amplifier_2/pha-202+_amplifier.kicad_sch (KiCad schematic)
At the start: 16 parts, among them J1 SMA, J2 SMA, J3 PWR, U1 PHA-202+

Commit message: h
Parts:
- removed H5: MountingHole_Pad, MountingHole:MountingHole_3.2mm_M3_DIN965_Pad_TopBottom, symbol Mechanical:MountingHole_Pad
- removed J3: PWR, Connector_PinHeader_2.54mm:PinHeader_1x02_P2.54mm_Vertical, symbol Connector_Generic:Conn_01x02
- added J3: PWR, TerminalBlock_Phoenix:TerminalBlock_Phoenix_MKDS-1,5-2_1x02_P5.00mm_Horizontal, symbol Connector:Screw_Terminal_01x02
- H1, H2, H3, H4: value MountingHole_Pad -> M2.5; footprint MountingHole:MountingHole_3.2mm_M3_DIN965_Pad_TopBottom -> MountingHole:MountingHole_2.7mm_M2.5_DIN965_Pad_TopBottom
Connections:
- net GND: now also J3.1 (Pin_1)
- net VCC: now also J3.2 (Pin_2)
Other:
- moved on the sheet: L1
