File: EBYTE-E28-2G4M27S-breakout/e28.kicad_pcb (KiCad board)
At the start: 2 copper layers, 30.6 x 29.7 mm, 10 parts, among them J1 Conn_01x08, J1 HDR-M-2.54_1x6, J2 Conn_01x08, J2 HDR-M-2.54_1x8, U1 E28-2G4M27S

Commit message: garbage
Parts:
- removed C11, C14: 10uF, e28:C1210
- removed C12: 100nF, e28:C0805
- removed the J1 at (137.3, 110.0)
- removed the J2 at (162.7, 111.3)
- J1: renamed from J2; footprint Connector_PinHeader_2.54mm:PinHeader_1x06_P2.54mm_Vertical -> Connector_PinHeader_2.54mm:PinHeader_1x08_P2.54mm_Vertical; moved to B.Cu
- J2: renamed from J1; footprint Connector_PinHeader_2.54mm:PinHeader_1x06_P2.54mm_Vertical -> Connector_PinHeader_2.54mm:PinHeader_1x08_P2.54mm_Vertical; moved to B.Cu
- U1: value E28-2G4M27S -> ~; footprint e28:E28-2G4M20S -> E28-2G4M27S:E28-2G4M27S
- moved J2 47.3 mm to (161.5, 133.4)
- moved U1 23.7 mm to (150.1, 133.7)
- moved C2 20.8 mm to (153.9, 134.7), turned to 180 degrees
- moved C1 20.3 mm to (157.5, 134.7)
- moved J1 15.6 mm to (138.6, 115.6), turned to 180 degrees
Connections:
- J1 pad 2: RX_EN -> TX_EN
- J1 pad 3: NSS -> NRESET
- J1 pad 4: SCK -> BUSY
- J1 pad 5: MOSI -> DIO1
- J1 pad 6: MISO -> DIO2
- J2 pad 1: unconnected-(J1-Pin_1-Pad1) -> +3V3
- J2 pad 2: DIO3 -> MISO
- J2 pad 3: DIO2 -> MOSI
- J2 pad 4: DIO1 -> SCK
- J2 pad 5: BUSY -> NSS
- J2 pad 6: NRESET -> RX_EN
- U1 pad 1: 3V3 -> +3V3
- U1 pad 15: (no net) -> DIO3
Routing:
- net GND: track 82.8 -> 0.02 mm, vias 64 -> 63
- net 3V3: track 22.5 -> 0.00 mm, vias 1 -> 0
- net 5V: track 10.2 -> 0.00 mm
- net NSS: track 9.29 -> 3.97 mm
- net SCK: track 8.56 -> 3.44 mm
- net RX_EN: track 8.47 -> 3.97 mm
- net DIO3: track 0.00 -> 3.93 mm
- net TX_EN: track 8.46 -> 5.39 mm
- net MOSI: track 6.94 -> 3.89 mm
- net BUSY: track 7.78 -> 4.76 mm
- net NRESET: track 9.20 -> 6.23 mm
- net DIO1: track 6.51 -> 4.04 mm
- net DIO2: track 5.98 -> 3.52 mm
- net MISO: track 6.00 -> 4.49 mm
- added copper zone on F.Cu, net +3V3
Other:
- board size 30.6 x 29.7 mm -> 26 x 22 mm
- board text added: "E28-2G4M Breakout board"
- board text added: "GND GND RX_EN CS SCK MOSI MISO 3V3"
- board text added: "GND TX_EN RST BSY DIO1 DIO2 DIO3 GND"
- board text added: "MCzop 2025"
- board text added: "Rev. 1.1"
- board text removed: "5V"
- board text removed: "BUSY"
- board text removed: "DIO1"
- board text removed: "DIO2"
- board text removed: "G"
- board text removed: "MISO"
- board text removed: "MOSI"
- board text removed: "NC"
- board text removed: "NSS"
- board text removed: "RESET"
- board text removed: "RXEN"
- board text removed: "SCK"
- board text removed: "TXEN"
- board text removed: "V1.0 2020"
