File: EBYTE-E28-2G4M27S-breakout/e28.kicad_sch (KiCad schematic)
At the start: 5 parts, among them J1 Conn_01x08, J2 Conn_01x08

Commit message: garbage
Parts:
- J1: renamed from J2; footprint Connector_PinHeader_2.54mm:PinHeader_1x06_P2.54mm_Vertical -> Connector_PinHeader_2.54mm:PinHeader_1x08_P2.54mm_Vertical
- J2: renamed from J1; footprint Connector_PinHeader_2.54mm:PinHeader_1x06_P2.54mm_Vertical -> Connector_PinHeader_2.54mm:PinHeader_1x08_P2.54mm_Vertical
- U1: footprint (none) -> E28-2G4M27S:E28-2G4M27S
Connections:
- net +3V3: now also J2.1 (Pin_1); no longer J1.7 (Pin_7)
- net BUSY: now also J1.4 (Pin_4); no longer J2.5 (Pin_5)
- net DIO1: now also J1.5 (Pin_5); no longer J2.4 (Pin_4)
- net DIO2: now also J1.6 (Pin_6); no longer J2.3 (Pin_3)
- net DIO3: now also J1.7 (Pin_7); no longer J2.2 (Pin_2)
- net GND: now also J2.7 (Pin_7), J2.8 (Pin_8), U1.10 (GND)
- net MISO: now also J2.2 (Pin_2); no longer J1.6 (Pin_6)
- net MOSI: now also J2.3 (Pin_3); no longer J1.5 (Pin_5)
- net NRESET: now also J1.3 (Pin_3); no longer J2.6 (Pin_6)
- net NSS: now also J2.5 (Pin_5); no longer J1.3 (Pin_3)
- net RX_EN: now also J2.6 (Pin_6); no longer J1.2 (Pin_2)
- net SCK: now also J2.4 (Pin_4); no longer J1.4 (Pin_4)
- net TX_EN: now also J1.2 (Pin_2); no longer J2.7 (Pin_7)
