File: esp32s3wroom-devboard/esp32s3wroom-devboard.kicad_sch (KiCad schematic)
At the start: 27 parts, among them J1 USB C, J2 GPIO, J3 GPIO, SW1 BOOT, SW2 RST, U1 ESP32-S3-WROOM-1, U2 USBLC6-2SC6, U3 LDL1117S33R

Commit message: garbage
Parts:
- R7: value 33 -> 270
